Commit message: setup the basic environment and catkin_make

File: src/com760cw2_group16/urdf/group16Bot.urdf (robot description, URDF)
Before this commit: robot group16Bot, 2 links, 1 joints
Joints:
- joint base_to_laser: origin xyz=0 0 0.1 -> xyz=0 0 0.1 rpy=0 0 0

Commit message: Spawn random world - still failling to spawn robot

File: src/com760cw2_group16/urdf/group16Bot.urdf (robot description, URDF)
Before this commit: robot group16Bot, 2 links, 1 joints
Links:
- removed link laser
- link base_link: mass None -> 1.0; geometry collision box size=1 1 1; visual box size=1 1 1
Joints:
- removed joint base_to_laser

Commit message: spawn the robot   o Add Laser   o Add wheels

File: src/com760cw2_group16/urdf/group16Bot.urdf (robot description, URDF)
Before this commit: robot minimal_bot, 1 links, 0 joints
Links:
- added link dummy_base
- added link laser, mass 0.1; collision cylinder length=0.1 radius=0.05; visual cylinder length=0.1 radius=0.05
- added link left_wheel, mass 0.1; collision cylinder length=0.05 radius=0.05; visual cylinder length=0.05 radius=0.05
- added link right_wheel, mass 0.1; collision cylinder length=0.05 radius=0.05; visual cylinder length=0.05 radius=0.05
- link base_link: geometry collision box size=0.4 0.4 0.2; visual box size=0.4 0.4 0.2
Joints:
- added joint base_to_laser: type fixed, parent base_link, child laser, origin xyz=0 0 0.2 rpy=0 0 0
- added joint fixed_base_joint: type fixed, parent dummy_base, child base_link, origin xyz=0 0 0 rpy=0 0 0
- added joint left_wheel_joint: type continuous, parent base_link, child left_wheel, origin xyz=-0.2 0 -0.1 rpy=0 1.5708 0, axis 0 1 0
- added joint right_wheel_joint: type continuous, parent base_link, child right_wheel, origin xyz=0.2 0 -0.1 rpy=0 1.5708 0, axis 0 1 0

Commit message: add movement to robot

File: src/com760cw2_group16/urdf/group16Bot.urdf (robot description, URDF)
Before this commit: robot group16Bot, 5 links, 4 joints
Links:
- added link front_wheel, mass 0.05; collision cylinder length=0.03 radius=0.03; visual cylinder length=0.03 radius=0.03
Joints:
- added joint base_to_front_wheel: type fixed, parent base_link, child front_wheel, origin xyz=0 0.2 -0.1 rpy=0 1.5708 0

Commit message: Fix robot to have 4 wheels

File: src/com760cw2_group16/urdf/group16Bot.urdf (robot description, URDF)
Before this commit: robot group16Bot, 6 links, 5 joints
Links:
- removed link front_wheel
- removed link left_wheel
- removed link right_wheel
- added link left_wheel_back, mass 0.1; collision cylinder length=0.05 radius=0.05; visual cylinder length=0.05 radius=0.05
- added link left_wheel_front, mass 0.1; collision cylinder length=0.05 radius=0.05; visual cylinder length=0.05 radius=0.05
- added link right_wheel_back, mass 0.1; collision cylinder length=0.05 radius=0.05; visual cylinder length=0.05 radius=0.05
- added link right_wheel_front, mass 0.1; collision cylinder length=0.05 radius=0.05; visual cylinder length=0.05 radius=0.05
Joints:
- removed joint base_to_front_wheel
- added joint left_rear_joint: type fixed, parent base_link, child left_wheel_back, origin xyz=-0.2 -0.2 -0.1 rpy=0 1.5708 0
- added joint right_rear_joint: type fixed, parent base_link, child right_wheel_back, origin xyz=0.2 -0.2 -0.1 rpy=0 1.5708 0
- joint left_wheel_joint: child left_wheel -> left_wheel_front; origin xyz=-0.2 0 -0.1 rpy=0 1.5708 0 -> xyz=-0.2 0.2 -0.1 rpy=0 1.5708 0
- joint right_wheel_joint: child right_wheel -> right_wheel_front; origin xyz=0.2 0 -0.1 rpy=0 1.5708 0 -> xyz=0.2 0.2 -0.1 rpy=0 1.5708 0

Commit message: Complete Robot - moving

File: src/com760cw2_group16/urdf/group16Bot.urdf (robot description, URDF)
Before this commit: robot group16Bot, 7 links, 6 joints
Links:
- removed link base_link
- removed link dummy_base
- removed link left_wheel_back
- removed link left_wheel_front
- removed link right_wheel_back
- removed link right_wheel_front
- added link base_link_chassis, mass 5; collision box size=0.5 0.3 0.07; collision sphere radius=0.05
- added link left_wheel, mass 0.2; collision cylinder length=0.04 radius=0.1; visual cylinder length=0.04 radius=0.1
- added link right_wheel, mass 0.2; collision cylinder length=0.04 radius=0.1; visual cylinder length=0.04 radius=0.1
Joints:
- removed joint fixed_base_joint
- removed joint left_rear_joint
- removed joint left_wheel_joint
- removed joint right_rear_joint
- removed joint right_wheel_joint
- added joint left_wheel_hinge: type continuous, parent base_link_chassis, child left_wheel, origin xyz=-0.05 -0.15 0 rpy=0 0 0, axis 0 1 0, limit effort=10000 velocity=1000
- added joint right_wheel_hinge: type continuous, parent base_link_chassis, child right_wheel, origin xyz=-0.05 0.15 0 rpy=0 0 0, axis 0 1 0, limit effort=10000 velocity=1000
- joint base_to_laser: parent base_link -> base_link_chassis
