Commit message: Avoid obstacles and walls near start and target point

File: src/com760cw2_group16/urdf/4Willgroup16Bot.urdf (robot description, URDF)
Before this commit: robot group16Bot, 7 links, 6 joints
Links:
- removed link base_link
- removed link dummy_base
- added link base_link_chassis, mass 1.0; collision box size=0.4 0.4 0.2; visual box size=0.4 0.4 0.2
- link left_wheel_back: mass 0.1 -> 0.2; geometry collision cylinder length=0.04 radius=0.1; visual cylinder length=0.04 radius=0.1
- link left_wheel_front: mass 0.1 -> 0.2; geometry collision cylinder length=0.04 radius=0.1; visual cylinder length=0.04 radius=0.1
- link right_wheel_back: mass 0.1 -> 0.2; geometry collision cylinder length=0.04 radius=0.1; visual cylinder length=0.04 radius=0.1
- link right_wheel_front: mass 0.1 -> 0.2; geometry collision cylinder length=0.04 radius=0.1; visual cylinder length=0.04 radius=0.1
Joints:
- removed joint fixed_base_joint
- removed joint left_rear_joint
- removed joint left_wheel_joint
- removed joint right_rear_joint
- removed joint right_wheel_joint
- added joint left_wheel_back_hinge: type continuous, parent base_link_chassis, child left_wheel_back, origin xyz=-0.05 -0.25 -0.1 rpy=0 0 0, axis 0 1 0, limit effort=10000 velocity=1000
- added joint left_wheel_front_hinge: type continuous, parent base_link_chassis, child left_wheel_front, origin xyz=-0.05 -0.05 -0.1 rpy=0 0 0, axis 0 1 0, limit effort=10000 velocity=1000
- added joint right_wheel_back_hinge: type continuous, parent base_link_chassis, child right_wheel_back, origin xyz=-0.05 0.25 -0.1 rpy=0 0 0, axis 0 1 0, limit effort=10000 velocity=1000
- added joint right_wheel_front_hinge: type continuous, parent base_link_chassis, child right_wheel_front, origin xyz=-0.05 0.05 -0.1 rpy=0 0 0, axis 0 1 0, limit effort=10000 velocity=1000
- joint base_to_laser: origin xyz=0 0 0.2 rpy=0 0 0 -> xyz=0 0 0.1 rpy=0 0 0; parent base_link -> base_link_chassis

Commit message: add 4 wheels robot

File: src/com760cw2_group16/urdf/4Willgroup16Bot.urdf (robot description, URDF)
Before this commit: robot group16Bot, 6 links, 5 joints
Links:
- added link front_marker; visual box size=0.1 0.02 0.02
Joints:
- added joint front_marker_joint: type fixed, parent base_link_chassis, child front_marker, origin xyz=0 0 0 rpy=0 0 0
- joint base_to_laser: origin xyz=0 0 0.1 rpy=0 0 0 -> xyz=0 0 0.2 rpy=0 0 0
- joint left_wheel_back_hinge: origin xyz=-0.05 -0.25 -0.1 rpy=0 0 0 -> xyz=-0.1  0.15 -0.1 rpy=0 0 0
- joint left_wheel_front_hinge: origin xyz=-0.05 -0.05 -0.1 rpy=0 0 0 -> xyz=0.1  0.15 -0.1 rpy=0 0 0
- joint right_wheel_back_hinge: origin xyz=-0.05 0.25 -0.1 rpy=0 0 0 -> xyz=-0.1 -0.15 -0.1 rpy=0 0 0
- joint right_wheel_front_hinge: origin xyz=-0.05 0.05 -0.1 rpy=0 0 0 -> xyz=0.1 -0.15 -0.1 rpy=0 0 0
